File: stlinkv21_jlinkob/stlinkv21_jlinkob.kicad_pcb (KiCad board)
At the start: 2 copper layers, 50 x 25 mm, 32 parts, among them CON1 CORTEX-DEBUGGER_HOST, J1 USB_C, J2 Conn_01x02, J3 Conn_01x04, J4 Conn_02x05_Odd_Even, U1 STM32F103CBTx, U3 LM1117-3.3, Y1 Crystal_GND24_Small

Commit message: 20210214
Parts:
- C4, C6: footprint Capacitor_SMD:C_0603_1608Metric -> Capacitor_Tantalum_SMD:CP_EIA-7343-43_Kemet-X_Pad2.25x2.55mm_HandSolder
- RN1, RN2, RN3, RN4: footprint Resistor_SMD:R_Array_Concave_4x0603 -> mybays_connector:R_Array_4x0603_jump_0.2
- Y1: value Crystal_GND24_Small -> Crystal_Small; footprint Crystal:Crystal_SMD_3225-4Pin_3.2x2.5mm -> Crystal:Crystal_SMD_5032-2Pin_5.0x3.2mm
- moved C6 26.6 mm to (128.9, 97.2)
- moved C5 20.3 mm to (122.8, 95.2), turned to 90 degrees
- moved R5 8.87 mm to (102.6, 95.0)
- moved D3 6.99 mm to (102.6, 96.7), turned to 180 degrees
- moved C3 5.97 mm to (113.0, 78.5), turned to 90 degrees
- moved D1 3.68 mm to (141.3, 97.6), turned to 180 degrees
- moved R3 3.24 mm to (143.1, 96.0), turned to 180 degrees
- moved R4 3.02 mm to (136.6, 96.0)
- moved Y1 1.98 mm to (128.0, 86.4), turned to 90 degrees
- moved C1 1.56 mm to (125.2, 87.9), turned to 90 degrees
- moved C4 1.45 mm to (106.8, 78.2)
- moved D2 1.26 mm to (138.2, 97.6)
- moved C2 1.05 mm to (125.2, 84.8), turned to 270 degrees
- moved R2 0.80 mm to (116.2, 79.4)
Connections:
- CON1 pad 1: Net-(CON1-Pad1) -> VBUS
- J4 pad 1: Net-(J4-Pad1) -> VBUS
- Y1 pad 2: GND -> Net-(C2-Pad1)
Routing:
- net GND: track 13.5 -> 175.4 mm, vias 0 -> 11
- net +3V3: track 46.3 -> 167.3 mm, vias 0 -> 6
- net VBUS: track 18.2 -> 71.4 mm, vias 0 -> 1
- net PA9: track 0.00 -> 39.4 mm, vias 0 -> 2
- net PA3: track 0.00 -> 35.4 mm, vias 0 -> 3
- net PB6: track 0.00 -> 26.7 mm, vias 0 -> 1
- net PB13: track 0.00 -> 26.0 mm, vias 0 -> 1
- net PB14: track 2.34 -> 27.9 mm, vias 0 -> 1
- net TXD: track 0.00 -> 25.5 mm, vias 0 -> 2
- net PA4: track 0.00 -> 23.0 mm, vias 0 -> 2
- net RXD: track 0.08 -> 22.6 mm, vias 0 -> 2
- net SWDIO: track 0.00 -> 21.0 mm, vias 0 -> 3
- net SWCLK: track 0.00 -> 17.4 mm, vias 0 -> 1
- net SWO: track 0.00 -> 16.2 mm, vias 0 -> 1
- net RST: track 0.00 -> 14.9 mm, vias 0 -> 1
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- added copper zone on B.Cu, net GND
- added copper zone on F.Cu, net GND
Other:
- rule trace_min: 0.2 -> 0.1
- board text added: "1"
- board text added: "10"
- board text added: "2"
- board text added: "3"
- board text added: "3.3V"
- board text added: "4"
- board text added: "5"
- board text added: "5V"
- board text added: "6"
- board text added: "7"
- board text added: "8"
- board text added: "9"
- board text added: "GND"
- board text added: "Jlink-ob"
- board text added: "RST"
- board text added: "RXD"
- board text added: "SWCLK"
- board text added: "SWDIO"
- board text added: "SWO"
- board text added: "Stlink-V21"
- board text added: "TXD"
- board text removed: "jlink-ob"
- board text removed: "stlink-v21"
