File: stlinkv21_jlinkob/stlinkv21_jlinkob.kicad_pcb (KiCad board)
At the start: 2 copper layers, 50 x 25 mm, 32 parts, among them CON1 CORTEX-DEBUGGER_HOST, J1 USB_C, J2 Conn_01x02, J3 Conn_01x04, J4 Conn_02x05_Odd_Even, U1 STM32F103CBTx, U3 LM1117-3.3, Y1 Crystal_Small

Commit message: silk
Other:
- board text added: "3V3"
- board text added: "CLK"
- board text added: "DIO"
- board text added: "G"
