File: jlinkob_hs_5x5/connector.sch (KiCad schematic (older format))
At the start: 2 parts, among them J4 Conn_02x18_Odd_Even, J5 Conn_02x18_Odd_Even

Commit message: 20210818
Connections:
- net labels added: +3V3, GND, PA31, VCORE
Other:
- moved on the sheet: J5
