File: jlinkob_hs_5x5/debug_con.sch (KiCad schematic (older format))
At the start: 10 parts, among them CON2 CORTEX-DEBUGGER_HOST, J3 Conn_01x02, SW1 SW_Push

Commit message: 20210818
Connections:
- net GND: now also SW1.2
- net HOST_RESET: now reaches SW1.1
Changed lines of the file:
@@
 Text GLabel 1550 5300 0    50   Input ~ 0
 PA25
+$Comp
+L power:GND #PWR0134
+U 1 1 614544BA
+P 1900 4750
+F 0 "#PWR0134" H 1900 4500 50  0001 C CNN
+F 1 "GND" H 1905 4577 50  0000 C CNN
+F 2 "" H 1900 4750 50  0001 C CNN
+F 3 "" H 1900 4750 50  0001 C CNN
+	1    1900 4750
+	1    0    0    -1
+$EndComp
+Wire Wire Line
+	1900 4750 1900 4700
+Wire Wire Line
+	1450 4700 1500 4700
+Text GLabel 1450 4700 0    50   Input ~ 0
+HOST_RESET
 $EndSCHEMATC
