File: jlinkob_hs_5x5/jlinkob_hs.kicad_pcb (KiCad board)
At the start: 4 copper layers, 50 x 50 mm, 50 parts, among them CON1 CORTEX-DEBUGGER, CON2 CORTEX-DEBUGGER_HOST, J1 USB_C, J2 microusb, J3 Conn_01x02, J4 Conn_02x18_Odd_Even, J5 Conn_02x18_Odd_Even, SW1 SW_Push, U1 LM1117-3.3, Y1 12MHz

Commit message: 20210818
Parts:
- removed C20, C21, C22, C23, C24, C25: 100n, Capacitor_SMD:C_0402_1005Metric_Pad0.74x0.62mm_HandSolder
- removed D1: PRTR5V0U2X, Package_TO_SOT_SMD:SOT-143
- added Y2: Crystal, Crystal:Crystal_SMD_MicroCrystal_CC7V-T1A-2Pin_3.2x1.5mm_HandSoldering, F.Cu at (136.9, 66.9)
- C15, C16, C8, C9: moved to B.Cu
- C19: footprint Capacitor_SMD:C_0603_1608Metric_Pad1.08x0.95mm_HandSolder -> Capacitor_SMD:C_0402_1005Metric_Pad0.74x0.62mm_HandSolder
- TP1: footprint TestPoint:TestPoint_Pad_1.0x1.0mm -> mybays_connector:TestPoint_0.5
- U1: footprint Package_TO_SOT_SMD:SOT-223 -> Package_TO_SOT_SMD:SOT-223-3_TabPin2
- moved C18 51.5 mm to (114.0, 74.1), turned to 270 degrees
- moved C16 51.5 mm to (123.0, 80.0), turned to 90 degrees
- moved C9 49.3 mm to (120.0, 75.0)
- moved C11 48.5 mm to (118.5, 85.5), turned to 270 degrees
- moved C12 45.4 mm to (119.5, 85.5), turned to 270 degrees
- moved C14 45.3 mm to (119.8, 64.6), turned to 90 degrees
- moved C8 37.9 mm to (129.5, 80.0), turned to 90 degrees
- moved C13 32.4 mm to (110.3, 89.4), turned to 270 degrees
- moved C15 29.7 mm to (127.0, 64.6), turned to 90 degrees
- moved C26 29.7 mm to (106.9, 60.3), turned to 180 degrees
- moved R5 29.5 mm to (119.2, 90.8), turned to 180 degrees
- moved C5 29.3 mm to (131.1, 65.5), turned to 180 degrees
- moved C17 26.4 mm to (135.5, 77.0)
- moved R6 25.4 mm to (119.2, 88.8), turned to 180 degrees
- moved SW1 24.0 mm to (145.3, 68.2), turned to 270 degrees
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Connections:
- C27 pad 2: Net-(C27-Pad2) -> SHIELD
- J1 pad S1: Net-(C27-Pad2) -> SHIELD
- J2 pad 0: GND -> SHIELD
- J4 pad 1: (no net) -> GND
- J4 pad 2: (no net) -> GND
- J4 pad 33: (no net) -> PA0
- J4 pad 34: (no net) -> PA1
- J4 pad 35: (no net) -> GND
- J4 pad 36: (no net) -> GND
- J5 pad 1: (no net) -> GND
- J5 pad 10: PB21 -> PB17
- J5 pad 11: PB22 -> PB18
- J5 pad 12: PB23 -> PB19
- J5 pad 13: PB24 -> PB20
- J5 pad 14: PA12 -> PB21
- J5 pad 15: PA11 -> PB22
- J5 pad 16: PA10 -> PB23
- J5 pad 17: PA9 -> PB24
- J5 pad 18: PA8 -> PA12
- J5 pad 19: PA7 -> PA11
- J5 pad 2: (no net) -> GND
- J5 pad 20: PA6 -> PA10
- J5 pad 21: PA5 -> PA9
- J5 pad 22: PA4 -> PA8
- J5 pad 23: PA3 -> PA7
- J5 pad 24: PA2 -> PA6
- J5 pad 25: PA1 -> PA5
- J5 pad 26: PA0 -> PA4
- J5 pad 27: (no net) -> PA3
- J5 pad 28: (no net) -> PA2
- J5 pad 29: (no net) -> +3V3
- J5 pad 3: PB9 -> +3V3
- J5 pad 30: (no net) -> +3V3
- J5 pad 31: (no net) -> +3V3
- J5 pad 32: (no net) -> +3V3
- J5 pad 33: (no net) -> GND
- J5 pad 34: (no net) -> GND
- J5 pad 35: (no net) -> GND
- J5 pad 36: (no net) -> GND
- J5 pad 4: PB10 -> +3V3
- J5 pad 5: PB14 -> VCC
- J5 pad 6: PB17 -> PA31
- J5 pad 7: PB18 -> PB9
- J5 pad 8: PB19 -> PB10
- J5 pad 9: PB20 -> PB14
- R8 pad 2: Net-(C27-Pad2) -> SHIELD
- SW1 pad 1: (no net) -> HOST_RESET
- SW1 pad 2: (no net) -> GND
- U?.1 pad 49: (no net) -> Net-(U?.1-Pad49)
- U?.1 pad 50: (no net) -> Net-(U?.1-Pad50)
- U?.1 pad 86: (no net) -> PA31
Routing:
- net +3V3: track 0.00 -> 257.7 mm, vias 0 -> 7
- net GND: track 0.00 -> 119.7 mm, vias 0 -> 20
- net PA22: track 0.00 -> 61.5 mm
- net PA15: track 0.00 -> 53.8 mm, vias 0 -> 1
- net VCC: track 0.00 -> 51.3 mm, vias 0 -> 7
- net PA3: track 0.00 -> 49.8 mm, vias 0 -> 1
- net PA12: track 0.00 -> 45.7 mm, vias 0 -> 1
- net PA25: track 0.00 -> 43.1 mm, vias 0 -> 1
- net SHIELD: track 0.00 -> 41.5 mm
- net PA4: track 0.00 -> 40.4 mm, vias 0 -> 1
- net PA11: track 0.00 -> 40.2 mm, vias 0 -> 2
- net PA29: track 0.00 -> 40.0 mm, vias 0 -> 2
- net PA28: track 0.00 -> 39.6 mm, vias 0 -> 2
- net PA21: track 0.00 -> 37.9 mm
- net PA18: track 0.00 -> 37.3 mm, vias 0 -> 2
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- added copper zone on GND, net GND
- added copper zone on PWR, net VBUS
- added copper zone on PWR, net VCC
Other:
- net class Default: via_dia 0.8 -> 0.45; via_drill 0.4 -> 0.3
- rule via_min_size: 0.4 -> 0.45
- board text added: "3V3"
- board text added: "GND"
- board text added: "PA31"
- board text added: "VCORE"
